File: design/ACS.kicad_sch (KiCad schematic)
At the start: 83 parts, among them IC1 ADXL375BCCZ, IC2 I3G4250DTR, IC3 TPS56A37RPAR, IC4 74HCT126D,653, J1 SM06B-SRSS-TBLFSN, J2 XT30, J3 USB_C_Receptacle_USB2.0_14P, J4 SM04B-SRSS-TB, M1 Servo_W, M2 Servo_S, M3 Servo_E, M4 Servo_N, U1 STM32U575CGUx, U2 USBLC6-2SC6, U3 SN65HVD232, Y1 16MHz

Commit message: fix footprint assignment and add BOM
Parts:
- J1: footprint ACS:CONN_SM06B-SRSS-TB_JST -> footprints:CONN_SM06B-SRSS-TB_JST
- J2: footprint ACS:XT30 -> footprints:XT30
- J3: footprint Connector_USB:USB_C_Receptacle_Palconn_UTC16-G -> footprints:USB_C_Receptacle_Palconn_UTC16-G fixed
- J4: footprint ACS:CONN_SM04B-SRSS-TB_JST -> footprints:CONN_SM04B-SRSS-TB_JST
- TP1, TP2, TP3, TP4: footprint (none) -> TestPoint:TestPoint_Pad_D2.0mm
Changed lines of the file:
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@@
 			)
 		)
-		(property "Footprint" ""
+		(property "Footprint" "TestPoint:TestPoint_Pad_D2.0mm"
 			(at 29.21 116.84 0)
 			(effects
@@
 			)
 		)
-		(property "Footprint" ""
+		(property "Footprint" "TestPoint:TestPoint_Pad_D2.0mm"
 			(at 34.29 127 0)
 			(effects
@@
 			)
 		)
-		(property "Footprint" "ACS:CONN_SM04B-SRSS-TB_JST"
+		(property "Footprint" "footprints:CONN_SM04B-SRSS-TB_JST"
 			(at 350.012 206.248 0)
 			(effects
@@
 			)
 		)
-		(property "Footprint" "ACS:XT30"
+		(property "Footprint" "footprints:XT30"
 			(at 22.86 172.72 0)
 			(effects
@@
 			)
 		)
-		(property "Footprint" "ACS:CONN_SM06B-SRSS-TB_JST"
+		(property "Footprint" "footprints:CONN_SM06B-SRSS-TB_JST"
 			(at 261.62 252.73 0)
 			(effects
@@
 			)
 		)
-		(property "Footprint" ""
+		(property "Footprint" "TestPoint:TestPoint_Pad_D2.0mm"
 			(at 273.05 252.73 0)
 			(effects
@@
 			)
 		)
-		(property "Footprint" ""
+		(property "Footprint" "TestPoint:TestPoint_Pad_D2.0mm"
 			(at 25.4 186.69 0)
 			(effects
@@
 			)
 		)
-		(property "Footprint" "Connector_USB:USB_C_Receptacle_Palconn_UTC16-G"
+		(property "Footprint" "footprints:USB_C_Receptacle_Palconn_UTC16-G fixed"
 			(at 308.61 149.86 0)
 			(effects

Commit message: add gnd test
Parts:
- added TP5: TestPoint, TestPoint:TestPoint_Pad_D2.0mm, symbol Connector:TestPoint
Connections:
- net Earth: now also TP5.1
Changed lines of the file:
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@@
 	)
 	(junction
-		(at 232.41 203.2)
-		(diameter 0)
-		(color 0 0 0 0)
-	)
-	(junction
 		(at 102.87 133.35)
 		(diameter 0)
@@
 	)
 	(junction
+		(at 231.14 203.2)
+		(diameter 0)
+		(color 0 0 0 0)
+	)
+	(junction
 		(at 347.98 74.93)
 		(diameter 0)
@@
 	)
 	(junction
+		(at 233.68 203.2)
+		(diameter 0)
+		(color 0 0 0 0)
+	)
+	(junction
 		(at 116.84 195.58)
 		(diameter 0)
@@
 	(wire
 		(pts
-			(xy 232.41 203.2) (xy 233.68 203.2)
-		)
-		(stroke
-			(width 0)
-			(type default)
-		)
-	)
-	(wire
-		(pts
 			(xy 133.35 152.4) (xy 133.35 153.67)
 		)
@@
 	(wire
 		(pts
-			(xy 231.14 203.2) (xy 232.41 203.2)
+			(xy 231.14 203.2) (xy 233.68 203.2)
 		)
 		(stroke
@@
 	(wire
 		(pts
+			(xy 224.79 203.2) (xy 231.14 203.2)
+		)
+		(stroke
+			(width 0)
+			(type default)
+		)
+	)
+	(wire
+		(pts
 			(xy 322.58 152.4) (xy 336.55 152.4)
 		)
@@
 	)
 	(symbol
+		(lib_id "Connector:TestPoint")
+		(at 224.79 203.2 180)
+		(unit 1)
+		(exclude_from_sim no)
+		(in_bom yes)
+		(on_board yes)
+		(dnp no)
+		(property "Reference" "TP5"
+			(at 226.314 205.74 0)
+			(effects
+				(font
+					(size 1.27 1.27)
+				)
+				(justify right)
+			)
+		)
+		(property "Value" "TestPoint"
+			(at 226.314 208.28 0)
+			(effects
+				(font
+					(size 1.27 1.27)
+				)
+				(justify right)
+			)
+		)
+		(property "Footprint" "TestPoint:TestPoint_Pad_D2.0mm"
+			(at 219.71 203.2 0)
+			(effects
+				(font
+					(size 1.27 1.27)
+				)
+				(hide yes)
+			)
+		)
+		(property "Datasheet" "~"
+			(at 219.71 203.2 0)
+			(effects
+				(font
+					(size 1.27 1.27)
+				)
+				(hide yes)
+			)
+		)
+		(property "Description" "test point"
+			(at 224.79 203.2 0)
+			(effects
+				(font
+					(size 1.27 1.27)
+				)
+				(hide yes)
+			)
+		)
+		(pin "1"
+		)
+		(instances
+			(project "ACS"
+				(path "/7be06de6-fc21-4b76-a5c8-2a235dbbd876"
+					(reference "TP5")
+					(unit 1)
+				)
+			)
+		)
+	)
+	(symbol
 		(lib_id "power:Earth")
 		(at 33.02 83.82 0)
@@
 	(symbol
 		(lib_id "power:Earth")
-		(at 232.41 203.2 0)
+		(at 233.68 203.2 0)
 		(unit 1)
 		(exclude_from_sim no)
@@
 		(fields_autoplaced yes)
 		(property "Reference" "#PWR019"
-			(at 232.41 209.55 0)
+			(at 233.68 209.55 0)
 			(effects
 				(font
@@
 		)
 		(property "Value" "Earth"
-			(at 232.41 208.28 0)
+			(at 233.68 208.28 0)
 			(effects
 				(font
@@
 		)
 		(property "Footprint" ""
-			(at 232.41 203.2 0)
+			(at 233.68 203.2 0)
 			(effects
 				(font
@@
 		)
 		(property "Datasheet" "~"
-			(at 232.41 203.2 0)
+			(at 233.68 203.2 0)
 			(effects
 				(font
@@
 		)
 		(property "Description" "Power symbol creates a global label with name \"Earth\""
-			(at 232.41 203.2 0)
+			(at 233.68 203.2 0)
 			(effects
 				(font

Commit message: design review fixes
Connections:
- net Earth: now also J3.S1 (SHIELD)
- no-connect marks 25 -> 24
Other:
- note removed: "Should SHIELD be floating?"
Changed lines of the file:
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@@
-		)
-	)
-	(text "Should SHIELD \nbe floating?"
-		(exclude_from_sim no)
-		(at 294.894 176.784 0)
-		(effects
-			(font
-				(size 1.27 1.27)
-			)
 		)
 	)
@@
 	)
 	(junction
+		(at 304.8 172.72)
+		(diameter 0)
+		(color 0 0 0 0)
+	)
+	(junction
 		(at 153.67 99.06)
 		(diameter 0)
@@
 	)
 	(no_connect
-		(at 297.18 172.72)
-	)
-	(no_connect
 		(at 246.38 148.59)
 	)
@@
 		)
 		(stroke
+			(width 0)
+			(type default)
+		)
+	)
+	(wire
+		(pts
+			(xy 297.18 172.72) (xy 304.8 172.72)
+		)
+		(stroke

Commit message: design review fixes
Parts:
- removed C25, C26, C27, C28, C29: 4u7, SamacSys_Parts:CAPC0603X55N, symbol Device:C
- removed L2: 1u, SamacSys_Parts:INDC2012X105N, symbol Device:L_Small
- added C11: 22u, SamacSys_Parts:GRM18x, symbol Device:C
- added C28, C29, C35, C36, C37: 100n, SamacSys_Parts:CAPC0603X35N, symbol Device:C_Small
- renumbered C21 to C1, C22 to C10, C36 to C12, C1 to C13, C2 to C14, C37 to C15, C4 to C16, C6 to C17, C7 to C18, C3 to C19, C20 to C2, C8 to C20, C9 to C21, C5 to C22, C10 to C23, C11 to C24, C12 to C25, C13 to C26, C14 to C27, C31 to C3, C16 to C30, C17 to C31, C18 to C32, C15 to C33, C19 to C34, C30 to C38, C24 to C4, C23 to C5, C32 to C6, C33 to C7, C35 to C8, C34 to C9, F3 to F1, F1 to F2, F2 to F3, IC3 to IC2, IC2 to IC3, J2 to J1, J1 to J2, L3 to L2, R12 to R1, R5 to R10, R6 to R11, R7 to R12, R8 to R13, R9 to R14, R1 to R2, R10 to R3, R11 to R4, R14 to R5, R13 to R6, R2 to R7, R3 to R8, R4 to R9, TP3 to TP1, TP4 to TP2, TP2 to TP3, TP5 to TP4, TP1 to TP5
Connections:
- net +3V3: now also PS1.10 (VOUT_2), PS1.9 (VOUT_1), R3.2, C11.1; no longer C1.1, C10.1, IC1.1 (VDD_I/O), IC1.6 (VS), IC3.1 (VDDIO), IC3.15 (RES_6), IC3.16 (VDD)
- net +3V3A: now also C1.1, C10.1, IC1.1 (VDD_I/O), IC1.6 (VS), IC3.1 (VDDIO), IC3.15 (RES_6), IC3.16 (VDD)
- net +5V5: now also C28.1, C29.1, C35.2, C36.2, C37.2
- net Earth: now also C11.2, C28.2, C29.2, C35.1, C36.1, C37.1
Other:
- note added: "Add 100 nF capacitors to all A-pins"
